Commit message: 로봇: 몸통 카메라 렌즈 프레임(depth_camera_lens_link, +x 0.010 m) URDF 추가, eyes 수평 화각을 Dabai 깊이 67.9° 로

File: src/robot/map_vla_description/urdf/map_vla.urdf.xacro (robot description, xacro)
@@ -10,4 +10,22 @@
   <xacro:property name="arm_yaw" value="0.0"/>
   <xacro:omx_f prefix="omx_" />
+  <!-- ===== Body camera lens (Orbbec Dabai): depth_camera_link is the sensor BODY centre (collision box 0.02 m deep,
+       base_link x 0.074..0.094 = the camera panel of the limo_base mesh). The lens / optical centre is on the panel's
+       front face: +0.010 m along depth_camera_link x -> base_link (0.094, 0, 0.03). This is where the OmniGibson body
+       camera `eyes` sits (src/robot/og/limo_omx_source_config.yaml, robot-agent 391c04b) and what scenemap cam 0 /
+       FK tables must use (depth_link stays the upstream body-centre optical frame). -->
+  <joint name="depth_camera_lens_joint" type="fixed">
+    <parent link="depth_camera_link"/>
+    <child link="depth_camera_lens_link"/>
+    <origin xyz="0.010 0 0" rpy="0 0 0"/>
+  </joint>
+  <link name="depth_camera_lens_link"/>
+  <!-- optical frame: z forward, x right, y down (REP-103) -->
+  <joint name="depth_camera_lens_optical_joint" type="fixed">
+    <parent link="depth_camera_lens_link"/>
+    <child link="depth_camera_lens_optical_frame"/>
+    <origin xyz="0 0 0" rpy="-1.5707963 0 -1.5707963"/>
+  </joint>
+  <link name="depth_camera_lens_optical_frame"/>
   <joint name="omx_mount_joint" type="fixed">
     <parent link="base_link"/>

Commit message: 로봇: 잡는 점 프레임 grasp_point(omx_link5 x 0.08003 — E0 실측, OmniGibson get_eef_position, omx_end_effector_link 에서 손가락 축 0.0119 m 뒤) URDF 추가 — scenemap LIMO 순기구학 T_eef·잡기 규칙용

File: src/robot/map_vla_description/urdf/map_vla.urdf.xacro (robot description, xacro)
@@ -39,4 +39,14 @@
   </joint>
   <link name="omx_end_effector_link"/>
+  <!-- ===== Grasp point: where an object actually sits between the closed fingers (E0, robot-agent 66fe1ee,
+       docs/map_vla/CURRICULUM_BEHAVIOR2026.md 5.3; src/robot/og/e0/results/verify_eef_kp1e6.json get_eef_in_link5).
+       omx_link5 x = 0.08003, i.e. 0.0119 m behind omx_end_effector_link along the finger axis; same as OmniGibson
+       get_eef_position(). scenemap's LIMO grasp rule / FK tables (gen_limo_fk_table) use this frame. -->
+  <joint name="grasp_point_joint" type="fixed">
+    <parent link="omx_link5"/>
+    <child link="grasp_point"/>
+    <origin xyz="0.08003 -0.0016 0" rpy="0 0 0"/>
+  </joint>
+  <link name="grasp_point"/>
   <!-- ===== Manipulator wrist camera: the RGB camera already modelled in the OMX-F link5 mesh (no depth) =====
        The OMX-F mesh (follower_06_pan_Revised.stl, link5) contains a camera module. Pose measured from that mesh
